File: hardware/keeb.kicad_sch (KiCad schematic)
At the start: 6 parts, among them J1 USB_C_Receptacle_USB2.0, U1 STM32F103C8Tx

Commit message: feat: wip keyboard matrix and hardware changes
Parts:
- added D1, D10, D11, D12, D13, D14, D15, D16, D17, D18, D19, D2, D20, D21, D22, D23, D24, D25, D26, D27, D28, D29, D3, D30, D31, D32, D33, D34, D35, D36, D37, D38, D39, D4, D40, D41, D42, D43, D44, D45, D46, D47, D48, D49, D5, D50, D51, D52, D53, D54, D55, D56, D57, D58, D59, D6, D60, D61, D62, D63, D64, D65, D66, D67, D68, D69, D7, D70, D71, D72, D73, D74, D8, D9: D, symbol Device:D
- added H1, H2, H3, H4: MountingHole, symbol Mechanical:MountingHole
- added SW1: ESC, symbol Switch:SW_Push
- added SW10: F9, symbol Switch:SW_Push
- added SW11: F10, symbol Switch:SW_Push
- added SW12: F11, symbol Switch:SW_Push
- added SW13: F12, symbol Switch:SW_Push
- added SW14: Grave, symbol Switch:SW_Push
- added SW15: 1, symbol Switch:SW_Push
- added SW16: 2, symbol Switch:SW_Push
- added SW17: 3, symbol Switch:SW_Push
- added SW18: 4, symbol Switch:SW_Push
- added SW19: 5, symbol Switch:SW_Push
- added SW2: F1, symbol Switch:SW_Push
- added SW20: 6, symbol Switch:SW_Push
- added SW21: 7, symbol Switch:SW_Push
- added SW22: 8, symbol Switch:SW_Push
- added SW23: 9, symbol Switch:SW_Push
- added SW24: 0, symbol Switch:SW_Push
- added SW25: Minus, symbol Switch:SW_Push
- added SW26: Equal, symbol Switch:SW_Push
- added SW27: Backspace, symbol Switch:SW_Push
- added SW28: Tab, symbol Switch:SW_Push
- added SW29: Q, symbol Switch:SW_Push
- added SW3: F2, symbol Switch:SW_Push
- added SW30: W, symbol Switch:SW_Push
- added SW31: E, symbol Switch:SW_Push
- added SW32: R, symbol Switch:SW_Push
- added SW33: T, symbol Switch:SW_Push
- added SW34: Y, symbol Switch:SW_Push
- added SW35: U, symbol Switch:SW_Push
- added SW36: I, symbol Switch:SW_Push
- added SW37: O, symbol Switch:SW_Push
- added SW38: P, symbol Switch:SW_Push
- added SW39: LBracket, symbol Switch:SW_Push
- added SW4: F3, symbol Switch:SW_Push
- added SW40: RBracket, symbol Switch:SW_Push
- added SW41: Backslash, symbol Switch:SW_Push
- added SW42: Capslock, symbol Switch:SW_Push
- added SW43: A, symbol Switch:SW_Push
- added SW44: S, symbol Switch:SW_Push
- added SW45: D, symbol Switch:SW_Push
- added SW46: F, symbol Switch:SW_Push
- added SW47: G, symbol Switch:SW_Push
- added SW48: H, symbol Switch:SW_Push
- added SW49: J, symbol Switch:SW_Push
- added SW5: F4, symbol Switch:SW_Push
- added SW50: K, symbol Switch:SW_Push
- added SW51: L, symbol Switch:SW_Push
- added SW52: Semicolon, symbol Switch:SW_Push
- added SW53: Quote, symbol Switch:SW_Push
- added SW54: Enter, symbol Switch:SW_Push
- added SW55: LShift, symbol Switch:SW_Push
- added SW56: Z, symbol Switch:SW_Push
- added SW57: X, symbol Switch:SW_Push
- added SW58: C, symbol Switch:SW_Push
- added SW59: V, symbol Switch:SW_Push
- added SW6: F5, symbol Switch:SW_Push
- added SW60: B, symbol Switch:SW_Push
- added SW61: N, symbol Switch:SW_Push
- added SW62: M, symbol Switch:SW_Push
- added SW63: Comma, symbol Switch:SW_Push
- added SW64: Period, symbol Switch:SW_Push
- added SW65: Slash, symbol Switch:SW_Push
- added SW66: RShift, symbol Switch:SW_Push
- added SW67: LControl, symbol Switch:SW_Push
- added SW68, SW72: LGui, symbol Switch:SW_Push
- added SW69: LAlt, symbol Switch:SW_Push
- added SW7: F6, symbol Switch:SW_Push
- added SW70: Space, symbol Switch:SW_Push
- added SW71: RAlt, symbol Switch:SW_Push
- added SW73: Fn, symbol Switch:SW_Push
- added SW74: RControl, symbol Switch:SW_Push
- added SW75: Reset, Button_Switch_SMD:SW_MEC_5GSH9, symbol Switch:SW_Push
- added SW76: Boot, Button_Switch_SMD:SW_MEC_5GSH9, symbol Switch:SW_Push
- added SW8: F7, symbol Switch:SW_Push
- added SW9: F8, symbol Switch:SW_Push
- renumbered R3 to R1, R1 to R2, R2 to R3
Connections:
- net BOOT: now also SW76.1
- net RESET: now also SW75.1
- net ROW0: now reaches U1.10 (PA0)
- net ROW0: now also SW1.1, SW10.1, SW11.1, SW12.1, SW13.1, SW14.1, SW15.1, SW16.1, SW17.1, SW18.1, SW19.1, SW2.1, SW20.1, SW21.1, SW22.1, SW23.1, SW24.1, SW25.1, SW26.1, SW27.1, SW28.1, SW29.1, SW3.1, SW30.1, SW31.1, SW32.1, SW33.1, SW34.1, SW35.1, SW36.1, SW37.1, SW38.1, SW39.1, SW4.1, SW40.1, SW41.1, SW42.1, SW43.1, SW44.1, SW45.1, SW46.1, SW47.1, SW48.1, SW49.1, SW5.1, SW50.1, SW51.1, SW52.1, SW53.1, SW54.1, SW55.1, SW56.1, SW57.1, SW58.1, SW59.1, SW6.1, SW60.1, SW61.1, SW62.1, SW63.1, SW64.1, SW65.1, SW66.1, SW67.1, SW68.1, SW69.1, SW7.1, SW70.1, SW71.1, SW72.1, SW73.1, SW74.1, SW8.1, SW9.1
- net ROW1: now reaches U1.11 (PA1)
- net ROW2: now reaches U1.12 (PA2)
- net ROW3: now reaches U1.13 (PA3)
- net ROW4: now reaches U1.14 (PA4)
- net ROW5: now reaches U1.15 (PA5)
- net COL0: now reaches U1.18 (PB0)
- net COL0: now also D1.1 (K), D14.1 (K), D28.1 (K), D42.1 (K), D55.1 (K), D67.1 (K)
- net COL1: now reaches U1.19 (PB1)
- net COL1: now also D15.1 (K), D2.1 (K), D29.1 (K), D43.1 (K), D68.1 (K)
- net COL2: now reaches U1.20 (PB2)
- net COL2: now also D16.1 (K), D3.1 (K), D30.1 (K), D44.1 (K), D56.1 (K), D69.1 (K)
- net COL10: now reaches U1.21 (PB10)
- net COL10: now also D10.1 (K), D24.1 (K), D38.1 (K), D52.1 (K), D64.1 (K), D71.1 (K)
- net COL11: now reaches U1.22 (PB11)
- net COL11: now also D11.1 (K), D25.1 (K), D39.1 (K), D53.1 (K), D65.1 (K), D72.1 (K)
- net COL12: now reaches U1.25 (PB12)
- net COL12: now also D12.1 (K), D26.1 (K), D40.1 (K), D73.1 (K)
- net COL3: now reaches U1.39 (PB3)
- net COL3: now also D17.1 (K), D31.1 (K), D4.1 (K), D45.1 (K), D57.1 (K)
- net COL4: now reaches U1.40 (PB4)
- net COL4: now also D18.1 (K), D32.1 (K), D46.1 (K), D5.1 (K), D58.1 (K)
- net COL5: now reaches U1.41 (PB5)
- net COL5: now also D19.1 (K), D33.1 (K), D47.1 (K), D59.1 (K), D6.1 (K)
- net COL6: now reaches U1.42 (PB6)
- net COL6: now also D20.1 (K), D34.1 (K), D48.1 (K), D60.1 (K), D7.1 (K), D70.1 (K)
- net COL7: now reaches U1.43 (PB7)
- net COL7: now also D21.1 (K), D35.1 (K), D49.1 (K), D61.1 (K), D8.1 (K)
- net COL8: now reaches U1.45 (PB8)
- net COL8: now also D22.1 (K), D36.1 (K), D50.1 (K), D62.1 (K), D9.1 (K)
- net COL9: now reaches U1.46 (PB9)
- net COL9: now also D23.1 (K), D37.1 (K), D51.1 (K), D63.1 (K)
- net USB_D+ renamed USB_DP
- net USB_D- renamed USB_DM
- new net: D48.2 (A), SW48.2
- new net: D40.2 (A), SW40.2
- new net: D20.2 (A), SW20.2
- new net: D13.2 (A), SW13.2
- new net: D1.2 (A), SW1.2
- new net: D43.2 (A), SW43.2
- new net: D64.2 (A), SW64.2
- new net: D46.2 (A), SW46.2
- new net: D29.2 (A), SW29.2
- new net: D21.2 (A), SW21.2
- new net: D67.2 (A), SW67.2
- new net: D23.2 (A), SW23.2
- new net: D10.2 (A), SW10.2
- new net: D9.2 (A), SW9.2
- new net: D22.2 (A), SW22.2
- new net: D26.2 (A), SW26.2
- new net: D32.2 (A), SW32.2
- new net: D35.2 (A), SW35.2
- new net: D73.2 (A), SW73.2
- new net: D5.2 (A), SW5.2
- new net: D24.2 (A), SW24.2
- new net: D71.2 (A), SW71.2
- new net: D6.2 (A), SW6.2
- new net: D70.2 (A), SW70.2
- new net: D17.2 (A), SW17.2
- new net: D7.2 (A), SW7.2
- new net: D61.2 (A), SW61.2
- new net: D58.2 (A), SW58.2
- new net: D39.2 (A), SW39.2
- new net: D2.2 (A), SW2.2
- new net: D50.2 (A), SW50.2
- new net: D36.2 (A), SW36.2
- new net: D25.2 (A), SW25.2
- new net: D63.2 (A), SW63.2
- new net: D15.2 (A), SW15.2
- new net: D68.2 (A), SW68.2
- new net: D59.2 (A), SW59.2
- new net: D52.2 (A), SW52.2
- new net: D37.2 (A), SW37.2
- new net: D16.2 (A), SW16.2
- new net: D14.2 (A), SW14.2
- new net: D53.2 (A), SW53.2
- new net: D60.2 (A), SW60.2
- new net: D19.2 (A), SW19.2
- new net: D27.2 (A), SW27.2
- new net: D4.2 (A), SW4.2
- new net: D45.2 (A), SW45.2
- new net: D74.2 (A), SW74.2
- new net: D51.2 (A), SW51.2
- new net: D18.2 (A), SW18.2
- new net: D69.2 (A), SW69.2
- new net: D42.2 (A), SW42.2
- new net: D11.2 (A), SW11.2
- new net: D56.2 (A), SW56.2
- new net: D44.2 (A), SW44.2
- new net: D38.2 (A), SW38.2
- new net: D65.2 (A), SW65.2
- new net: D62.2 (A), SW62.2
- new net: D28.2 (A), SW28.2
- new net: D47.2 (A), SW47.2
- new net: D49.2 (A), SW49.2
- new net: D30.2 (A), SW30.2
- new net: D41.2 (A), SW41.2
- new net: D3.2 (A), SW3.2
- new net: D12.2 (A), SW12.2
- new net: D54.2 (A), SW54.2
- new net: D8.2 (A), SW8.2
- new net: D34.2 (A), SW34.2
- new net: D31.2 (A), SW31.2
- new net: D72.2 (A), SW72.2
- new net: D55.2 (A), SW55.2
- new net: D66.2 (A), SW66.2
- new net: D33.2 (A), SW33.2
- new net: D57.2 (A), SW57.2
- new net COL13: D13.1 (K), D27.1 (K), D41.1 (K), D54.1 (K), D66.1 (K), D74.1 (K)
Other:
- removed sheet Matrix
- moved on the sheet: C1, J1, R1, R2, R3

Commit message: refactor: change default layout
Forgot arrow keys, added power regulator and some others
Parts:
- removed C1: 0.1uF, symbol Device:C
- removed H1, H2, H3, H4: MountingHole, symbol Mechanical:MountingHole
- removed R1: 100K, symbol Device:R
- added C2, C3: 1uF, Capacitor_SMD:C_0201_0603Metric, symbol Device:C
- added C4, C5: 30pF, Capacitor_SMD:C_0201_0603Metric, symbol Device:C_Small
- added D75, D76: D, Diode_SMD:D_0201_0603Metric, symbol Device:D
- added D77: Schottky 5819W, Diode_SMD:D_0603_1608Metric, symbol Device:D_Schottky
- added F1: TLC_PSMD0050, Fuse:Fuse_0603_1608Metric, symbol Device:Fuse
- added FB1: 100@100MHz, Inductor_SMD:L_0603_1608Metric, symbol Device:FerriteBead
- added SW75: Down, Button_Switch_Keyboard:SW_Cherry_MX_1.00u_PCB, symbol Switch:SW_Push
- added SW76: Right, Button_Switch_Keyboard:SW_Cherry_MX_1.00u_PCB, symbol Switch:SW_Push
- added U2: XC6206PxxxMR, Package_TO_SOT_SMD:SOT-23-3, symbol Regulator_Linear:XC6206PxxxMR
- added Y1: 12MHz-20pF, Crystal:Crystal_SMD_0603-4Pin_6.0x3.5mm, symbol Device:Crystal_GND24_Small
- D1, D10, D11, D12, D13, D14, D15, D16, D17, D18, D19, D2, D20, D21, D22, D23, D24, D25, D26, D27, D28, D29, D3, D30, D31, D32, D33, D34, D35, D36, D37, D38, D39, D4, D40, D41, D42, D43, D44, D45, D46, D47, D48, D49, D5, D50, D51, D52, D53, D54, D55, D56, D57, D58, D59, D6, D60, D61, D62, D63, D64, D65, D66, D67, D68, D69, D7, D70, D71, D72, D73, D74, D8, D9: footprint (none) -> Diode_SMD:D_0201_0603Metric
- R2, R3: value 5.1K -> 5.11K; footprint (none) -> Resistor_SMD:R_0603_1608Metric
- SW1, SW10, SW11, SW12, SW13, SW14, SW15, SW16, SW17, SW18, SW19, SW2, SW20, SW21, SW22, SW23, SW24, SW25, SW26, SW29, SW3, SW30, SW31, SW32, SW33, SW34, SW35, SW36, SW37, SW38, SW39, SW4, SW40, SW41, SW43, SW44, SW45, SW46, SW47, SW48, SW49, SW5, SW50, SW51, SW52, SW53, SW56, SW57, SW58, SW59, SW6, SW60, SW61, SW62, SW63, SW64, SW65, SW67, SW68, SW69, SW7, SW71, SW72, SW73, SW8, SW9: footprint (none) -> Button_Switch_Keyboard:SW_Cherry_MX_1.00u_PCB
- SW27, SW28: footprint (none) -> Button_Switch_Keyboard:SW_Cherry_MX_1.50u_PCB
- SW42, SW54: footprint (none) -> Button_Switch_Keyboard:SW_Cherry_MX_1.75u_PCB
- SW55: footprint (none) -> Button_Switch_Keyboard:SW_Cherry_MX_2.00u_PCB
- SW66: value RShift -> Up; footprint (none) -> Button_Switch_Keyboard:SW_Cherry_MX_1.00u_PCB
- SW70: footprint (none) -> Button_Switch_Keyboard:SW_Cherry_MX_6.25u_PCB
- SW74: value RControl -> Left; footprint (none) -> Button_Switch_Keyboard:SW_Cherry_MX_1.00u_PCB
- renumbered SW75 to SW77, SW76 to SW78
Connections:
- net +3.3V: now also C3.1, U2.2 (VO)
- net COL10: now also D73.1 (K); no longer D71.1 (K)
- net COL11: now also D74.1 (K); no longer D72.1 (K)
- net COL12: now also D54.1 (K), D66.1 (K), D75.1 (K); no longer D73.1 (K)
- net COL13: now also D76.1 (K); no longer D54.1 (K), D66.1 (K), D74.1 (K)
- net COL5: now also D70.1 (K)
- net COL6: no longer D7.1 (K), D70.1 (K)
- net COL7: now also D7.1 (K); no longer D8.1 (K)
- net COL8: now also D71.1 (K), D8.1 (K); no longer D9.1 (K)
- net COL9: now also D72.1 (K), D9.1 (K)
- net GND: now also C2.2, C3.2, C4.2, C5.2, U2.1 (GND), Y1.2, Y1.4
- net OSC_IN: now also C4.1, Y1.3
- net OSC_OUT: now also C5.1, Y1.1
- net ROW0: no longer SW14.1, SW15.1, SW16.1, SW17.1, SW18.1, SW19.1, SW20.1, SW21.1, SW22.1, SW23.1, SW24.1, SW25.1, SW26.1, SW27.1, SW28.1, SW29.1, SW30.1, SW31.1, SW32.1, SW33.1, SW34.1, SW35.1, SW36.1, SW37.1, SW38.1, SW39.1, SW40.1, SW41.1, SW42.1, SW43.1, SW44.1, SW45.1, SW46.1, SW47.1, SW48.1, SW49.1, SW50.1, SW51.1, SW52.1, SW53.1, SW54.1, SW55.1, SW56.1, SW57.1, SW58.1, SW59.1, SW60.1, SW61.1, SW62.1, SW63.1, SW64.1, SW65.1, SW66.1, SW67.1, SW68.1, SW69.1, SW70.1, SW71.1, SW72.1, SW73.1, SW74.1
- net ROW1: now also SW14.1, SW15.1, SW16.1, SW17.1, SW18.1, SW19.1, SW20.1, SW21.1, SW22.1, SW23.1, SW24.1, SW25.1, SW26.1, SW27.1
- net ROW2: now also SW28.1, SW29.1, SW30.1, SW31.1, SW32.1, SW33.1, SW34.1, SW35.1, SW36.1, SW37.1, SW38.1, SW39.1, SW40.1, SW41.1
- net ROW3: now also SW42.1, SW43.1, SW44.1, SW45.1, SW46.1, SW47.1, SW48.1, SW49.1, SW50.1, SW51.1, SW52.1, SW53.1, SW54.1
- net ROW4: now also SW55.1, SW56.1, SW57.1, SW58.1, SW59.1, SW60.1, SW61.1, SW62.1, SW63.1, SW64.1, SW65.1, SW66.1
- net ROW5: now also SW67.1, SW68.1, SW69.1, SW70.1, SW71.1, SW72.1, SW73.1, SW74.1, SW75.1, SW76.1
- net VBUS: now also D77.2 (A)
- new net: D77.1 (K), F1.1
- new net: D75.2 (A), SW75.2
- new net: D76.2 (A), SW76.2
- new net: F1.2, FB1.1
- new net +5V: C2.1, FB1.2, U2.3 (VI)
- no-connect marks 2 -> 14
Other:
- moved on the sheet: R2, R3
